File: kicad/location_sensors.kicad_sch (KiCad schematic)
At the start: 24 parts

Commit message: Fixed up or explained all DRC violations.
Parts:
- renumbered R8 to R11, R9 to R12, R10 to R13, R11 to R14, R12 to R15, R13 to R16, R14 to R17, R15 to R18
Changed lines of the file:
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@@
 		(dnp no)
 		(fields_autoplaced yes)
-		(property "Reference" "R13"
+		(property "Reference" "R16"
 			(at 210.82 132.0799 0)
 			(effects
@@
 			(project "tv_slider"
 				(path "/914c4b67-a7a4-47f3-8515-668040fd3f8c/816aa5cb-6066-4d97-997e-6fcfac1c1c32"
-					(reference "R13")
+					(reference "R16")
 					(unit 1)
 				)
@@
 		(dnp no)
 		(fields_autoplaced yes)
-		(property "Reference" "R10"
+		(property "Reference" "R13"
 			(at 87.63 55.88 90)
 			(effects
@@
 			(project ""
 				(path "/914c4b67-a7a4-47f3-8515-668040fd3f8c/816aa5cb-6066-4d97-997e-6fcfac1c1c32"
-					(reference "R10")
+					(reference "R13")
 					(unit 1)
 				)
@@
 		(dnp no)
 		(fields_autoplaced yes)
-		(property "Reference" "R12"
+		(property "Reference" "R15"
 			(at 106.68 132.0799 0)
 			(effects
@@
 			(project "tv_slider"
 				(path "/914c4b67-a7a4-47f3-8515-668040fd3f8c/816aa5cb-6066-4d97-997e-6fcfac1c1c32"
-					(reference "R12")
+					(reference "R15")
 					(unit 1)
 				)
@@
 		(dnp no)
 		(fields_autoplaced yes)
-		(property "Reference" "#PWR066"
+		(property "Reference" "#PWR067"
 			(at 213.36 106.68 0)
 			(effects
@@
 			(project ""
 				(path "/914c4b67-a7a4-47f3-8515-668040fd3f8c/816aa5cb-6066-4d97-997e-6fcfac1c1c32"
-					(reference "#PWR066")
+					(reference "#PWR067")
 					(unit 1)
 				)
@@
 		(dnp no)
 		(fields_autoplaced yes)
-		(property "Reference" "R9"
+		(property "Reference" "R12"
 			(at 210.82 54.6099 0)
 			(effects
@@
 			(project "tv_slider"
 				(path "/914c4b67-a7a4-47f3-8515-668040fd3f8c/816aa5cb-6066-4d97-997e-6fcfac1c1c32"
-					(reference "R9")
+					(reference "R12")
 					(unit 1)
 				)
@@
 		(dnp no)
 		(fields_autoplaced yes)
-		(property "Reference" "#PWR055"
+		(property "Reference" "#PWR056"
 			(at 109.22 29.21 0)
 			(effects
@@
 			(project ""
 				(path "/914c4b67-a7a4-47f3-8515-668040fd3f8c/816aa5cb-6066-4d97-997e-6fcfac1c1c32"
-					(reference "#PWR055")
+					(reference "#PWR056")
 					(unit 1)
 				)
@@
 		(dnp no)
 		(fields_autoplaced yes)
-		(property "Reference" "#PWR068"
+		(property "Reference" "#PWR069"
 			(at 187.96 120.65 0)
 			(effects
@@
 			(project "tv_slider"
 				(path "/914c4b67-a7a4-47f3-8515-668040fd3f8c/816aa5cb-6066-4d97-997e-6fcfac1c1c32"
-					(reference "#PWR068")
+					(reference "#PWR069")
 					(unit 1)
 				)
@@
 		(dnp no)
 		(fields_autoplaced yes)
-		(property "Reference" "#PWR057"
+		(property "Reference" "#PWR058"
 			(at 83.82 43.18 0)
 			(effects
@@
 			(project "tv_slider"
 				(path "/914c4b67-a7a4-47f3-8515-668040fd3f8c/816aa5cb-6066-4d97-997e-6fcfac1c1c32"
-					(reference "#PWR057")
+					(reference "#PWR058")
 					(unit 1)
 				)
@@
 		(dnp no)
 		(fields_autoplaced yes)
-		(property "Reference" "#PWR064"
+		(property "Reference" "#PWR065"
 			(at 208.28 81.28 0)
 			(effects
@@
 			(project "tv_slider"
 				(path "/914c4b67-a7a4-47f3-8515-668040fd3f8c/816aa5cb-6066-4d97-997e-6fcfac1c1c32"
-					(reference "#PWR064")
+					(reference "#PWR065")
 					(unit 1)
 				)
@@
 		(dnp no)
 		(fields_autoplaced yes)
-		(property "Reference" "#PWR067"
+		(property "Reference" "#PWR068"
 			(at 83.82 120.65 0)
 			(effects
@@
 			(project "tv_slider"
 				(path "/914c4b67-a7a4-47f3-8515-668040fd3f8c/816aa5cb-6066-4d97-997e-6fcfac1c1c32"
-					(reference "#PWR067")
+					(reference "#PWR068")
 					(unit 1)
 				)
@@
 		(dnp no)
 		(fields_autoplaced yes)
-		(property "Reference" "R15"
+		(property "Reference" "R18"
 			(at 191.77 133.35 90)
 			(effects
@@
 			(project "tv_slider"
 				(path "/914c4b67-a7a4-47f3-8515-668040fd3f8c/816aa5cb-6066-4d97-997e-6fcfac1c1c32"
-					(reference "R15")
+					(reference "R18")
 					(unit 1)
 				)
@@
 		(dnp no)
 		(fields_autoplaced yes)
-		(property "Reference" "#PWR058"
+		(property "Reference" "#PWR059"
 			(at 187.96 43.18 0)
 			(effects
@@
 			(project "tv_slider"
 				(path "/914c4b67-a7a4-47f3-8515-668040fd3f8c/816aa5cb-6066-4d97-997e-6fcfac1c1c32"
-					(reference "#PWR058")
+					(reference "#PWR059")
 					(unit 1)
 				)
@@
 		(dnp no)
 		(fields_autoplaced yes)
-		(property "Reference" "#PWR061"
+		(property "Reference" "#PWR062"
 			(at 93.98 81.28 0)
 			(effects
@@
 			(project ""
 				(path "/914c4b67-a7a4-47f3-8515-668040fd3f8c/816aa5cb-6066-4d97-997e-6fcfac1c1c32"
-					(reference "#PWR061")
+					(reference "#PWR062")
 					(unit 1)
 				)
@@
 		(dnp no)
 		(fields_autoplaced yes)
-		(property "Reference" "#PWR062"
+		(property "Reference" "#PWR063"
 			(at 104.14 81.28 0)
 			(effects
@@
 			(project "tv_slider"
 				(path "/914c4b67-a7a4-47f3-8515-668040fd3f8c/816aa5cb-6066-4d97-997e-6fcfac1c1c32"
-					(reference "#PWR062")
+					(reference "#PWR063")
 					(unit 1)
 				)
@@
 		(dnp no)
 		(fields_autoplaced yes)
-		(property "Reference" "#PWR063"
+		(property "Reference" "#PWR064"
 			(at 198.12 81.28 0)
 			(effects
@@
 			(project "tv_slider"
 				(path "/914c4b67-a7a4-47f3-8515-668040fd3f8c/816aa5cb-6066-4d97-997e-6fcfac1c1c32"
-					(reference "#PWR063")
+					(reference "#PWR064")
 					(unit 1)
 				)
@@
 		(dnp no)
 		(fields_autoplaced yes)
-		(property "Reference" "R14"
+		(property "Reference" "R17"
 			(at 87.63 133.35 90)
 			(effects
@@
 			(project "tv_slider"
 				(path "/914c4b67-a7a4-47f3-8515-668040fd3f8c/816aa5cb-6066-4d97-997e-6fcfac1c1c32"
-					(reference "R14")
+					(reference "R17")
 					(unit 1)
 				)
@@
 		(dnp no)
 		(fields_autoplaced yes)
-		(property "Reference" "R8"
+		(property "Reference" "R11"
 			(at 106.68 54.6099 0)
 			(effects
@@
 			(project "tv_slider"
 				(path "/914c4b67-a7a4-47f3-8515-668040fd3f8c/816aa5cb-6066-4d97-997e-6fcfac1c1c32"
-					(reference "R8")
+					(reference "R11")
 					(unit 1)
 				)
@@
 		(dnp no)
 		(fields_autoplaced yes)
-		(property "Reference" "#PWR069"
+		(property "Reference" "#PWR070"
 			(at 104.14 130.81 0)
 			(effects
@@
 			(project "tv_slider"
 				(path "/914c4b67-a7a4-47f3-8515-668040fd3f8c/816aa5cb-6066-4d97-997e-6fcfac1c1c32"
-					(reference "#PWR069")
+					(reference "#PWR070")
 					(unit 1)
 				)
@@
 		(dnp no)
 		(fields_autoplaced yes)
-		(property "Reference" "#PWR073"
+		(property "Reference" "#PWR074"
 			(at 198.12 158.75 0)
 			(effects
@@
 			(project "tv_slider"
 				(path "/914c4b67-a7a4-47f3-8515-668040fd3f8c/816aa5cb-6066-4d97-997e-6fcfac1c1c32"
-					(reference "#PWR073")
+					(reference "#PWR074")
 					(unit 1)
 				)
@@
 		(dnp no)
 		(fields_autoplaced yes)
-		(property "Reference" "#PWR072"
+		(property "Reference" "#PWR073"
 			(at 104.14 158.75 0)
 			(effects
@@
 			(project "tv_slider"
 				(path "/914c4b67-a7a4-47f3-8515-668040fd3f8c/816aa5cb-6066-4d97-997e-6fcfac1c1c32"
-					(reference "#PWR072")
+					(reference "#PWR073")
 					(unit 1)
 				)
@@
 		(dnp no)
 		(fields_autoplaced yes)
-		(property "Reference" "#PWR065"
+		(property "Reference" "#PWR066"
 			(at 109.22 106.68 0)
 			(effects
@@
 			(project ""
 				(path "/914c4b67-a7a4-47f3-8515-668040fd3f8c/816aa5cb-6066-4d97-997e-6fcfac1c1c32"
-					(reference "#PWR065")
+					(reference "#PWR066")
 					(unit 1)
 				)
@@
 		(dnp no)
 		(fields_autoplaced yes)
-		(property "Reference" "#PWR059"
+		(property "Reference" "#PWR060"
 			(at 104.14 53.34 0)
 			(effects
@@
 			(project ""
 				(path "/914c4b67-a7a4-47f3-8515-668040fd3f8c/816aa5cb-6066-4d97-997e-6fcfac1c1c32"
-					(reference "#PWR059")
+					(reference "#PWR060")
 					(unit 1)
 				)
@@
 		(dnp no)
 		(fields_autoplaced yes)
-		(property "Reference" "#PWR071"
+		(property "Reference" "#PWR072"
 			(at 93.98 158.75 0)
 			(effects
@@
 			(project "tv_slider"
 				(path "/914c4b67-a7a4-47f3-8515-668040fd3f8c/816aa5cb-6066-4d97-997e-6fcfac1c1c32"
-					(reference "#PWR071")
+					(reference "#PWR072")
 					(unit 1)
 				)
@@
 		(dnp no)
 		(fields_autoplaced yes)
-		(property "Reference" "#PWR070"
+		(property "Reference" "#PWR071"
 			(at 208.28 130.81 0)
 			(effects
@@
 			(project "tv_slider"
 				(path "/914c4b67-a7a4-47f3-8515-668040fd3f8c/816aa5cb-6066-4d97-997e-6fcfac1c1c32"
-					(reference "#PWR070")
+					(reference "#PWR071")
 					(unit 1)
 				)
@@
 		(dnp no)
 		(fields_autoplaced yes)
-		(property "Reference" "R11"
+		(property "Reference" "R14"
 			(at 191.77 55.88 90)
 			(effects
@@
 			(project "tv_slider"
 				(path "/914c4b67-a7a4-47f3-8515-668040fd3f8c/816aa5cb-6066-4d97-997e-6fcfac1c1c32"
-					(reference "R11")
+					(reference "R14")
 					(unit 1)
 				)
@@
 		(dnp no)
 		(fields_autoplaced yes)
-		(property "Reference" "#PWR056"
+		(property "Reference" "#PWR057"
 			(at 213.36 29.21 0)
 			(effects
@@
 			(project ""
 				(path "/914c4b67-a7a4-47f3-8515-668040fd3f8c/816aa5cb-6066-4d97-997e-6fcfac1c1c32"
-					(reference "#PWR056")
+					(reference "#PWR057")
 					(unit 1)
 				)
@@
 		(dnp no)
 		(fields_autoplaced yes)
-		(property "Reference" "#PWR060"
+		(property "Reference" "#PWR061"
 			(at 208.28 53.34 0)
 			(effects
@@
 			(project "tv_slider"
 				(path "/914c4b67-a7a4-47f3-8515-668040fd3f8c/816aa5cb-6066-4d97-997e-6fcfac1c1c32"
-					(reference "#PWR060")
+					(reference "#PWR061")
 					(unit 1)
 				)
@@
 		(dnp no)
 		(fields_autoplaced yes)
-		(property "Reference" "#PWR074"
+		(property "Reference" "#PWR075"
 			(at 208.28 158.75 0)
 			(effects
@@
 			(project "tv_slider"
 				(path "/914c4b67-a7a4-47f3-8515-668040fd3f8c/816aa5cb-6066-4d97-997e-6fcfac1c1c32"
-					(reference "#PWR074")
+					(reference "#PWR075")
 					(unit 1)
 				)

Commit message: Supplying the ESP32-C6-DEVKIT with 5V and using its 3V3 output to supply the boards logic. Removed the 3V3 switch mode power supply on the board.
Parts:
- renumbered C25 to C20, C26 to C21, C27 to C22, C28 to C23, C29 to C24, C30 to C25, C31 to C26, C32 to C27, D2 to D3, D3 to D4, D4 to D5, D5 to D6, R12 to R10, R13 to R11, R14 to R12, R15 to R13, R16 to R14, R17 to R15, R18 to R16, R11 to R9

Commit message: Updated to use more of JCLPCB's basic components. Added extra field "FT Rotation Offset" to get the correct orientation for placement at JCLPCB.
Parts:
- C20, C21, C24, C25: Dielectric X7R -> (none); LCSC (none) -> C14663; MF Murata -> Yageo; MP GRM188R72A104KA35D -> CC0603KRX7R9BB104; SupplierPN 490-3285-1-ND -> 311-1344-1-ND; Voltage 100V -> 50V
- C22, C23, C26, C27: Dielectric X7R -> (none); LCSC (none) -> C21122; MF Murata -> Samsung; MP GRM188R72A223KAC4J -> CL10B223KB8NNNC; SupplierPN 490-GRM188R72A223KAC4JCT-ND -> 1276-1104-1-ND; Voltage 100V -> 50V
- D3, D4, D5, D6: value SMF5V0A -> SMF5.0A; footprint Diode_SMD:D_SMF -> Diode_SMD:D_SOD-123F; LCSC (none) -> C19077497; MF Vishay -> Hong Jiacheng; MP SMF5V0A-E3-08 -> SMF5.0A; SupplierPN SMF5V0A-E3-08CT-ND -> 1655-SMF5.0ACT-ND
- FB1, FB2, FB3, FB4: LCSC (none) -> C1015; MF Murata -> Sunlord; MP BLM21PG221SN1D -> GZ2012D101TF
- R10, R13, R14, R9: LCSC (none) -> C23162; MF Yageo -> Uni Royal; MP RC0603FR-074K7L -> 0603WAF4701T5E
- R11, R12, R15, R16: LCSC (none) -> C21190; MF Yageo -> Uni Royal; MP RC0603FR-071KL -> 0603WAF1001T5E
