File: kicad/motor_drive.kicad_sch (KiCad schematic)
At the start: 10 parts, among them U5 DRV8452SPWPR

Commit message: Reviewed the ESP32-C6-DEVKIT GPIO's. Some of them have a dual function and are better left untouched.
Connections:
- net ENABLE is gone; now on net +3V3: U5.25 (ENABLE)
Changed lines of the file:
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@@
+	(wire
+		(pts
+			(xy 113.03 40.64) (xy 113.03 68.58)
+		)
+		(stroke
+			(width 0)
+			(type default)
+		)
+	)
 	(wire
 		(pts
@@
 	(wire
 		(pts
-			(xy 88.9 68.58) (xy 116.84 68.58)
-		)
-		(stroke
-			(width 0)
-			(type default)
-		)
-	)
-	(wire
-		(pts
 			(xy 208.28 54.61) (xy 208.28 91.44)
 		)
@@
 		(pts
 			(xy 88.9 83.82) (xy 116.84 83.82)
+		)
+		(stroke
+			(width 0)
+			(type default)
+		)
+	)
+	(wire
+		(pts
+			(xy 113.03 68.58) (xy 116.84 68.58)
 		)
 		(stroke
@@
 			)
 			(justify left)
-		)
-	)
-	(hierarchical_label "ENABLE"
-		(shape input)
-		(at 88.9 68.58 180)
-		(effects
-			(font
-				(size 1.27 1.27)
-			)
-			(justify right)
 		)
 	)
@@
 					(unit 1)
 				)
+			)
+		)
+	)
+	(symbol
+		(lib_id "power:+3V3")
+		(at 113.03 40.64 0)
+		(unit 1)
+		(exclude_from_sim no)
+		(in_bom yes)
+		(on_board yes)
+		(dnp no)
+		(fields_autoplaced yes)
+		(property "Reference" "#PWR097"
+			(at 113.03 44.45 0)
+			(effects
+				(font
+					(size 1.27 1.27)
+				)
+				(hide yes)
+			)
+		)
+		(property "Value" "+3V3"
+			(at 113.03 35.56 0)
+			(effects
+				(font
+					(size 1.27 1.27)
+				)
+			)
+		)
+		(property "Footprint" ""
+			(at 113.03 40.64 0)
+			(effects
+				(font
+					(size 1.27 1.27)
+				)
+				(hide yes)
+			)
+		)
+		(property "Datasheet" ""
+			(at 113.03 40.64 0)
+			(effects
+				(font
+					(size 1.27 1.27)
+				)
+				(hide yes)
+			)
+		)
+		(property "Description" "Power symbol creates a global label with name \"+3V3\""
+			(at 113.03 40.64 0)
+			(effects
+				(font
+					(size 1.27 1.27)
+				)
+				(hide yes)
+			)
+		)
+		(pin "1"
+		)
+		(instances
+			(project "tv_slider"
+				(path "/914c4b67-a7a4-47f3-8515-668040fd3f8c/e5516eed-629d-4c0b-bb03-2e43d030d802"
+					(reference "#PWR097")
+					(unit 1)
+				)

Commit message: Supplying the ESP32-C6-DEVKIT with 5V and using its 3V3 output to supply the boards logic. Removed the 3V3 switch mode power supply on the board.
Parts:
- renumbered C17 to C12, C18 to C13, C19 to C14, C20 to C15, C21 to C16, C22 to C17, C23 to C18, C24 to C19, R10 to R8, U5 to U4
Changed lines of the file:
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@@
 		(dnp no)
 		(fields_autoplaced yes)
-		(property "Reference" "U5"
+		(property "Reference" "U4"
 			(at 137.16 38.1 0)
 			(effects
@@
 			(project ""
 				(path "/914c4b67-a7a4-47f3-8515-668040fd3f8c/e5516eed-629d-4c0b-bb03-2e43d030d802"
-					(reference "U5")
+					(reference "U4")
 					(unit 1)
 				)
@@
 		(dnp no)
 		(fields_autoplaced yes)
-		(property "Reference" "#PWR049"
+		(property "Reference" "#PWR045"
 			(at 161.29 129.54 0)
 			(effects
@@
 			(project ""
 				(path "/914c4b67-a7a4-47f3-8515-668040fd3f8c/e5516eed-629d-4c0b-bb03-2e43d030d802"
-					(reference "#PWR049")
+					(reference "#PWR045")
 					(unit 1)
 				)
@@
 		(dnp no)
 		(fields_autoplaced yes)
-		(property "Reference" "#PWR054"
+		(property "Reference" "#PWR050"
 			(at 232.41 129.54 0)
 			(effects
@@
 			(project "tv_slider"
 				(path "/914c4b67-a7a4-47f3-8515-668040fd3f8c/e5516eed-629d-4c0b-bb03-2e43d030d802"
-					(reference "#PWR054")
+					(reference "#PWR050")
 					(unit 1)
 				)
@@
 		(dnp no)
 		(fields_autoplaced yes)
-		(property "Reference" "C23"
+		(property "Reference" "C18"
 			(at 236.22 114.6809 0)
 			(effects
@@
 			(project "tv_slider"
 				(path "/914c4b67-a7a4-47f3-8515-668040fd3f8c/e5516eed-629d-4c0b-bb03-2e43d030d802"
-					(reference "C23")
+					(reference "C18")
 					(unit 1)
 				)
@@
 		(on_board yes)
 		(dnp no)
-		(property "Reference" "#PWR042"
+		(property "Reference" "#PWR038"
 			(at 175.26 44.45 0)
 			(effects
@@
 			(project "tv_slider"
 				(path "/914c4b67-a7a4-47f3-8515-668040fd3f8c/e5516eed-629d-4c0b-bb03-2e43d030d802"
-					(reference "#PWR042")
+					(reference "#PWR038")
 					(unit 1)
 				)
@@
 		(on_board yes)
 		(dnp no)
-		(property "Reference" "#PWR045"
+		(property "Reference" "#PWR041"
 			(at 205.74 114.3 0)
 			(effects
@@
 			(project "tv_slider"
 				(path "/914c4b67-a7a4-47f3-8515-668040fd3f8c/e5516eed-629d-4c0b-bb03-2e43d030d802"
-					(reference "#PWR045")
+					(reference "#PWR041")
 					(unit 1)
 				)
@@
 		(dnp no)
 		(fields_autoplaced yes)
-		(property "Reference" "#PWR043"
+		(property "Reference" "#PWR039"
 			(at 208.28 44.45 0)
 			(effects
@@
 			(project "tv_slider"
 				(path "/914c4b67-a7a4-47f3-8515-668040fd3f8c/e5516eed-629d-4c0b-bb03-2e43d030d802"
-					(reference "#PWR043")
+					(reference "#PWR039")
 					(unit 1)
 				)
@@
 		(dnp no)
 		(fields_autoplaced yes)
-		(property "Reference" "#PWR097"
+		(property "Reference" "#PWR035"
 			(at 113.03 44.45 0)
 			(effects
@@
 			(project "tv_slider"
 				(path "/914c4b67-a7a4-47f3-8515-668040fd3f8c/e5516eed-629d-4c0b-bb03-2e43d030d802"
-					(reference "#PWR097")
+					(reference "#PWR035")
 					(unit 1)
 				)
@@
 		(dnp no)
 		(fields_autoplaced yes)
-		(property "Reference" "C17"
+		(property "Reference" "C12"
 			(at 179.07 49.5299 0)
 			(effects
@@
 			(project "tv_slider"
 				(path "/914c4b67-a7a4-47f3-8515-668040fd3f8c/e5516eed-629d-4c0b-bb03-2e43d030d802"
-					(reference "C17")
+					(reference "C12")
 					(unit 1)
 				)
@@
 		(on_board yes)
 		(dnp no)
-		(property "Reference" "C19"
+		(property "Reference" "C14"
 			(at 180.34 115.5699 0)
 			(effects
@@
 			(project "tv_slider"
 				(path "/914c4b67-a7a4-47f3-8515-668040fd3f8c/e5516eed-629d-4c0b-bb03-2e43d030d802"
-					(reference "C19")
+					(reference "C14")
 					(unit 1)
 				)
@@
 		(dnp no)
 		(fields_autoplaced yes)
-		(property "Reference" "#PWR052"
+		(property "Reference" "#PWR048"
 			(at 205.74 129.54 0)
 			(effects
@@
 			(project "tv_slider"
 				(path "/914c4b67-a7a4-47f3-8515-668040fd3f8c/e5516eed-629d-4c0b-bb03-2e43d030d802"
-					(reference "#PWR052")
+					(reference "#PWR048")
 					(unit 1)
 				)
@@
 		(dnp no)
 		(fields_autoplaced yes)
-		(property "Reference" "#PWR050"
+		(property "Reference" "#PWR046"
 			(at 176.53 129.54 0)
 			(effects
@@
 			(project "tv_slider"
 				(path "/914c4b67-a7a4-47f3-8515-668040fd3f8c/e5516eed-629d-4c0b-bb03-2e43d030d802"
-					(reference "#PWR050")
+					(reference "#PWR046")
 					(unit 1)
 				)
@@
 		(dnp no)
 		(fields_autoplaced yes)
-		(property "Reference" "C20"
+		(property "Reference" "C15"
 			(at 195.58 115.5699 0)
 			(effects
@@
 			(project ""
 				(path "/914c4b67-a7a4-47f3-8515-668040fd3f8c/e5516eed-629d-4c0b-bb03-2e43d030d802"
-					(reference "C20")
+					(reference "C15")
 					(unit 1)
 				)
@@
 		(dnp no)
 		(fields_autoplaced yes)
-		(property "Reference" "#PWR040"
+		(property "Reference" "#PWR036"
 			(at 160.02 44.45 0)
 			(effects
@@
 			(project ""
 				(path "/914c4b67-a7a4-47f3-8515-668040fd3f8c/e5516eed-629d-4c0b-bb03-2e43d030d802"
-					(reference "#PWR040")
+					(reference "#PWR036")
 					(unit 1)
 				)
@@
 		(on_board yes)
 		(dnp no)
-		(property "Reference" "#PWR047"
+		(property "Reference" "#PWR043"
 			(at 232.41 114.3 0)
 			(effects
@@
 			(project "tv_slider"
 				(path "/914c4b67-a7a4-47f3-8515-668040fd3f8c/e5516eed-629d-4c0b-bb03-2e43d030d802"
-					(reference "#PWR047")
+					(reference "#PWR043")
 					(unit 1)
 				)
@@
 		(on_board yes)
 		(dnp no)
-		(property "Reference" "#PWR046"
+		(property "Reference" "#PWR042"
 			(at 218.44 114.3 0)
 			(effects
@@
 			(project "tv_slider"
 				(path "/914c4b67-a7a4-47f3-8515-668040fd3f8c/e5516eed-629d-4c0b-bb03-2e43d030d802"
-					(reference "#PWR046")
+					(reference "#PWR042")
 					(unit 1)
 				)
@@
 		(on_board yes)
 		(dnp no)
-		(property "Reference" "#PWR048"
+		(property "Reference" "#PWR044"
 			(at 246.38 114.3 0)
 			(effects
@@
 			(project "tv_slider"
 				(path "/914c4b67-a7a4-47f3-8515-668040fd3f8c/e5516eed-629d-4c0b-bb03-2e43d030d802"
-					(reference "#PWR048")
+					(reference "#PWR044")
 					(unit 1)
 				)
@@
 		(dnp no)
 		(fields_autoplaced yes)
-		(property "Reference" "C21"
+		(property "Reference" "C16"
 			(at 209.55 115.5699 0)
 			(effects
@@
 			(project "tv_slider"
 				(path "/914c4b67-a7a4-47f3-8515-668040fd3f8c/e5516eed-629d-4c0b-bb03-2e43d030d802"
-					(reference "C21")
+					(reference "C16")
 					(unit 1)
 				)
@@
 		(dnp no)
 		(fields_autoplaced yes)
-		(property "Reference" "C22"
+		(property "Reference" "C17"
 			(at 222.25 115.5699 0)
 			(effects
@@
 			(project "tv_slider"
 				(path "/914c4b67-a7a4-47f3-8515-668040fd3f8c/e5516eed-629d-4c0b-bb03-2e43d030d802"
-					(reference "C22")
+					(reference "C17")
 					(unit 1)
 				)
@@
 		(dnp no)
 		(fields_autoplaced yes)
-		(property "Reference" "#PWR053"
+		(property "Reference" "#PWR049"
 			(at 218.44 129.54 0)
 			(effects
@@
 			(project "tv_slider"
 				(path "/914c4b67-a7a4-47f3-8515-668040fd3f8c/e5516eed-629d-4c0b-bb03-2e43d030d802"
-					(reference "#PWR053")
+					(reference "#PWR049")
 					(unit 1)
 				)
@@
 		(dnp no)
 		(fields_autoplaced yes)
-		(property "Reference" "R10"
+		(property "Reference" "R8"
 			(at 210.82 49.5299 0)
 			(effects
@@
 			(project "tv_slider"
 				(path "/914c4b67-a7a4-47f3-8515-668040fd3f8c/e5516eed-629d-4c0b-bb03-2e43d030d802"
-					(reference "R10")
+					(reference "R8")
 					(unit 1)
 				)
@@
 		(dnp no)
 		(fields_autoplaced yes)
-		(property "Reference" "#PWR051"
+		(property "Reference" "#PWR047"
 			(at 191.77 129.54 0)
 			(effects
@@
 			(project "tv_slider"
 				(path "/914c4b67-a7a4-47f3-8515-668040fd3f8c/e5516eed-629d-4c0b-bb03-2e43d030d802"
-					(reference "#PWR051")
+					(reference "#PWR047")
 					(unit 1)
 				)
@@
 		(on_board yes)
 		(dnp no)
-		(property "Reference" "#PWR041"
+		(property "Reference" "#PWR037"
 			(at 167.64 44.45 0)
 			(effects
@@
 			(project ""
 				(path "/914c4b67-a7a4-47f3-8515-668040fd3f8c/e5516eed-629d-4c0b-bb03-2e43d030d802"
-					(reference "#PWR041")
+					(reference "#PWR037")
 					(unit 1)
 				)
@@
 		(dnp no)
 		(fields_autoplaced yes)
-		(property "Reference" "C24"
+		(property "Reference" "C19"
 			(at 250.19 114.6809 0)
 			(effects
@@
 			(project "tv_slider"
 				(path "/914c4b67-a7a4-47f3-8515-668040fd3f8c/e5516eed-629d-4c0b-bb03-2e43d030d802"
-					(reference "C24")
+					(reference "C19")
 					(unit 1)
 				)
@@
 		(dnp no)
 		(fields_autoplaced yes)
-		(property "Reference" "#PWR044"
+		(property "Reference" "#PWR040"
 			(at 176.53 114.3 0)
 			(effects
@@
 			(project "tv_slider"
 				(path "/914c4b67-a7a4-47f3-8515-668040fd3f8c/e5516eed-629d-4c0b-bb03-2e43d030d802"
-					(reference "#PWR044")
+					(reference "#PWR040")
 					(unit 1)
 				)
@@
 		(dnp no)
 		(fields_autoplaced yes)
-		(property "Reference" "#PWR055"
+		(property "Reference" "#PWR051"
 			(at 246.38 129.54 0)
 			(effects
@@
 			(project "tv_slider"
 				(path "/914c4b67-a7a4-47f3-8515-668040fd3f8c/e5516eed-629d-4c0b-bb03-2e43d030d802"
-					(reference "#PWR055")
+					(reference "#PWR051")
 					(unit 1)
 				)
@@
 		(on_board yes)
 		(dnp no)
-		(property "Reference" "C18"
+		(property "Reference" "C13"
 			(at 179.07 60.9599 0)
 			(effects
@@
 			(project "tv_slider"
 				(path "/914c4b67-a7a4-47f3-8515-668040fd3f8c/e5516eed-629d-4c0b-bb03-2e43d030d802"
-					(reference "C18")
-					(unit 1)
-				)
+					(reference "C13")
+					(unit 1)
+				)

Commit message: Updated to use more of JCLPCB's basic components. Added extra field "FT Rotation Offset" to get the correct orientation for placement at JCLPCB.
Parts:
- C12, C15: Dielectric X7S -> (none); LCSC (none) -> C28323; MF Murata -> Samsung; MP GRM21BC72A105KE01L -> CL21B105KBFNNNE; SupplierPN 490-14464-1-ND -> 1276-1029-1-ND; Voltage 100V -> 50V
- C13, C14: Dielectric X7R -> (none); LCSC (none) -> C14663; MF Murata -> Yageo; MP GRM188R72A104KA35D -> CC0603KRX7R9BB104; SupplierPN 490-3285-1-ND -> 311-1344-1-ND; Voltage 100V -> 50V
- C16, C17: Dielectric X7R -> (none); LCSC (none) -> C57112; MF Murata -> Knowles Novacap; MP GRM188R72A103KA01D -> 0603B103K500NT; SupplierPN 490-GRM188R72A103KA01DCT-ND -> 1763-0603B103K500NTCT-ND; Voltage 100V -> 50V
- C18, C19: FT Rotation Offset (none) -> 180; LCSC (none) -> C1517667
- R8: LCSC (none) -> C25804; MF Yageo -> Uni Royal; MP RC0603FR-0710KL -> 0603WAF1002T5E
- U4: LCSC (none) -> C32469576

Commit message: Fixed rotation for JLCPCB.
Parts:
- U4: FT Rotation Offset (none) -> 270
Changed lines of the file:
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@@
 			)
 		)
-		(property "FT Rotation Offset" ""
+		(property "FT Rotation Offset" "270"
 			(at 137.16 73.66 0)
 			(effects
